File: loaf.kicad_sch (KiCad schematic)
At the start: 99 parts, among them J1 USB_C_Receptacle_USB2.0, J2 AVR-ISP-6, J3 OLED, SW1 SW_Push, SW10 SW_Push, SW11 SW_Push, SW12 SW_Push, SW13 SW_Push, SW14 SW_Push, SW15 SW_Push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

Commit message: switch diodes to sod-123
Parts:
- D10, D11, D12, D13, D14, D15, D16, D17, D18, D19, D20, D21, D22, D23, D24, D25, D26, D27, D28, D29, D3, D30, D31, D32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: footprint Diode_SMD:D_0805_2012Metric -> Diode_SMD:D_SOD-123
